File: dac_adc_pmod.kicad_pcb (KiCad board)
At the start: 2 copper layers, 20.3 x 48.3 mm, 24 parts, among them J1 pmod, J2 Analog, U1 LTC2627, U2 LTC2402

Commit message: fixed block capacitor
Routing:
- net +3V3: track 121.4 -> 107.8 mm, vias 2 -> 3
- net GND: track 91.8 -> 94.2 mm
- net /ldac: track 44.1 -> 45.6 mm
- net Net-(R5-Pad2): track 6.71 -> 7.26 mm
