File: dac_adc_pmod.kicad_sch (KiCad schematic)
At the start: 24 parts, among them J1 pmod, J2 Analog, U1 LTC2627, U2 LTC2402

Commit message: add screenshots
Other:
- company: (none) -> S59MZ
- title: (none) -> PMOD for DAC-ADC Loop
